File: PCBDesign/1.4Fv3/1.4Fv3.sch (EAGLE design)
At the start: 180 parts, among them U1 SN74LVC, U10 ISO7241, U11 PAM2305, U12 SN6501, U13 TRANSFO_3.3, U14 ADE9078, U15 PS2505, U16 SN74LVC, U17 PS2505, U2 PS2505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

Commit message: Schematic update
Parts:
- removed C11, C12, C21, C28, C30, C43, C46, C47: 22n, Nizanlib:0402-CAP
- R11, R12, R19, R20, R26, R27: value 1k -> 2k
- R14, R22, R41, R56, R57, R60, R68, R69: value 100 -> 0
- R16, R18, R42, R43, R54, R55, R66, R67: value 5 -> 20
- R36, R37, R58, R59, R63, R64, R65, R72: value 750k -> 245k
- R38, R39, R40, R44, R45, R46, R47, R48, R49, R50, R51, R75: value 400k -> 120k
Connections:
- net AGND: no longer C11.1, C12.2, C21.1, C28.2, C30.1, C43.2, C46.1, C47.2
- net N$2: no longer C21.2
- net N$24: no longer C30.2
- net N$27: no longer C28.1
- net N$3: no longer C43.1
- net N$48: no longer C11.2
- net N$56: no longer C12.1
- net N$7: no longer C46.2
- net N$8: no longer C47.1
Other:
- note added: "Date: 3/22/2019 3:17 PM"
- note added: "Math: For P = 80% for a 20% overvoltage head room, R_total for 208 = 366k R_total for 408 = 850k"
- note added: "Math: Input AC voltage should be scaled down to be less than the max of 0.707 Vrms Datasheet recommends a max of 50% of 0.707 Vrms in case of overvoltage But increasing the percent allows for better accuracy (Allows more output codes) Formula of determining resistance: R = [ (Input*1000) / (P% * 0.707) ] - 1000, where Input is either 208 or 480 and P% is scaled according to user perferred accurac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"
- note added: "Note: CT used that was used for testing was the AcuCT - H100 - 50 Split CT. At rated current of 50A, voltage output is expected to be 0.333 Vac at 200 Amps which should below the reccommended differential ADC input of 0.3535 Vrms. The CT needs a burden resistance of 10 Ohm. The following circuit is for CT usuage ONLY. For Rog. coil, refer to ADE9078 circuit for current sensing with coils. When me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"
- note added: "Note: Jumper settings allow for multiple 3-phase Delta and Wye service configurations as well as Blondel and non-Blondel metering strategies. Jumper settings is safe in testing, but maybe unsafe in general service as drawn. See release notes for jumper setting details."
- note added: "University of California, Irvine v.1.4Fv3 (c) 2018"
- note removed: "Date: 12/6/2018 12:05 PM"
- note removed: "Note: CT used that was used for testing was the AcuCT - H100 - 50 Split CT. At rated current of 50A, voltage output is expected to be 0.333 Vac at 200 Amps which should below the reccommended differential ADC input of 0.3535 Vrms. The CT needs a burden resistance of 10 Ohm. Use burden resistors as half-value pairs as specified by the CT used for R10/R11, R29/R30, R36/R37, R6/R7 For example, a 10 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"
- note removed: "Note: With the 480 Vac service option and an 50% overhead for overvoltage event, the max expected differential ADC input is 0.3535 Vrms. With the 208 Vac service option and an 50% overhead for overvoltage event, the max expected differential ADC input is 0.3535 Vrms Jumper settings allow for multiple 3-phase Delta and Wye service configurations as well as Blondel and non-Blondel metering strategi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"
- note removed: "University of California, Irvine v.1.2F (c) 2018"
