File: PCBDesign/1.4Fv3/1.4Fv4.brd (EAGLE design)
At the start: 87.6 x 57.1 mm, 180 parts, among them U1 SN74LVC, U10 ISO7241, U11 PAM2305, U12 SN6501, U13 TRANSFO_3.3, U14 ADE9078, U15 PS2505, U16 SN74LVC, U17 PS2505, U2 PS2505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

Commit message: Push up schematic with changes
Routing:
- net N$61: track 2.75 -> 0.99 mm
- net N$118: track 2.75 -> 0.99 mm
Changed lines of the file:
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@@
 <contactref element="R80" pad="2"/>
 <contactref element="R81" pad="1"/>
-<contactref element="J3" pad="1"/>
 <via x="5.08" y="46.99" extent="1-16" drill="0.35"/>
 <wire x1="3.344" y1="48.26" x2="4.614" y2="46.99" width="0.1524" layer="1"/>
@@
 <wire x1="8.89" y1="50.8" x2="5.08" y2="46.99" width="0.1524" layer="16"/>
 <via x="13.97" y="52.07" extent="1-16" drill="0.35"/>
-<wire x1="14.097" y1="54.61" x2="13.97" y2="54.483" width="0.1524" layer="1"/>
 <wire x1="13.97" y1="54.483" x2="13.97" y2="52.07" width="0.1524" layer="1"/>
 <wire x1="13.97" y1="52.07" x2="11.43" y2="52.07" width="0.1524" layer="16"/>
@@
 <via x="28.5994" y="48.26" extent="1-16" drill="0.35"/>
 <wire x1="28.5994" y1="48.26" x2="26.67" y2="48.26" width="0.1524" layer="1"/>
+<contactref element="J3" pad="1"/>
+<wire x1="13.97" y1="54.483" x2="14.097" y2="54.61" width="0" layer="19" extent="1-1"/>
 </signal>
 <signal name="GNDI">
@@
 <signal name="N$61">
 <contactref element="D3" pad="1"/>
+<wire x1="74.43" y1="37.4" x2="73.73" y2="38.1" width="0.1524" layer="1"/>
 <contactref element="R12" pad="1"/>
-<wire x1="74.43" y1="37.4" x2="73.73" y2="38.1" width="0.1524" layer="1"/>
-<wire x1="73.73" y1="38.1" x2="71.97" y2="38.1" width="0.1524" layer="1"/>
+<wire x1="71.97" y1="38.1" x2="73.73" y2="38.1" width="0" layer="19" extent="1-1"/>
 </signal>
 <signal name="N$118">
 <contactref element="D4" pad="1"/>
+<wire x1="74.43" y1="31.05" x2="73.73" y2="31.75" width="0.1524" layer="1"/>
 <contactref element="R20" pad="1"/>
-<wire x1="74.43" y1="31.05" x2="73.73" y2="31.75" width="0.1524" layer="1"/>
-<wire x1="73.73" y1="31.75" x2="71.97" y2="31.75" width="0.1524" layer="1"/>
+<wire x1="71.97" y1="31.75" x2="73.73" y2="31.75" width="0" layer="19" extent="1-1"/>
 </signal>
 <signal name="N$121">

Commit message: Changed resistor values 0->100
Parts:
- R14, R22, R41, R56, R57, R60, R68, R69: value 0 -> 100
Changed lines of the file:
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@@
 <attribute name="PROD_ID" value=" " x="8.89" y="27.94" size="1.778" layer="27" rot="R270" display="off"/>
 </element>
-<element name="R14" library="SparkFun-Resistors" library_urn="urn:adsk.eagle:library:532" package="0603" package3d_urn="urn:adsk.eagle:package:39650/1" value=" 0" x="10.16" y="19.05" smashed="yes">
+<element name="R14" library="SparkFun-Resistors" library_urn="urn:adsk.eagle:library:532" package="0603" package3d_urn="urn:adsk.eagle:package:39650/1" value=" 100" x="10.16" y="19.05" smashed="yes">
 <attribute name="NAME" x="9.652" y="18.288" size="0.6096" layer="21" font="vector" ratio="13" rot="R180" align="bottom-center"/>
 <attribute name="PROD_ID" value=" " x="10.16" y="19.05" size="1.778" layer="27" display="off"/>
@@
 <attribute name="PROD_ID" value=" " x="17.78" y="22.86" size="1.778" layer="27" display="off"/>
 </element>
-<element name="R22" library="SparkFun-Resistors" library_urn="urn:adsk.eagle:library:532" package="0603" package3d_urn="urn:adsk.eagle:package:39650/1" value=" 0" x="13.97" y="22.86" smashed="yes">
+<element name="R22" library="SparkFun-Resistors" library_urn="urn:adsk.eagle:library:532" package="0603" package3d_urn="urn:adsk.eagle:package:39650/1" value=" 100" x="13.97" y="22.86" smashed="yes">
 <attribute name="NAME" x="13.462" y="23.622" size="0.6096" layer="21" font="vector" ratio="13" align="bottom-center"/>
 <attribute name="PROD_ID" value=" " x="13.97" y="22.86" size="1.778" layer="27" display="off"/>
@@
 <attribute name="PROD_ID" value=" " x="21.59" y="17.78" size="1.778" layer="27" display="off"/>
 </element>
-<element name="R41" library="SparkFun-Resistors" library_urn="urn:adsk.eagle:library:532" package="0603" package3d_urn="urn:adsk.eagle:package:39650/1" value=" 0" x="10.16" y="13.97" smashed="yes">
+<element name="R41" library="SparkFun-Resistors" library_urn="urn:adsk.eagle:library:532" package="0603" package3d_urn="urn:adsk.eagle:package:39650/1" value=" 100" x="10.16" y="13.97" smashed="yes">
 <attribute name="NAME" x="9.652" y="13.208" size="0.6096" layer="21" font="vector" ratio="13" rot="R180" align="bottom-center"/>
 <attribute name="PROD_ID" value=" " x="10.16" y="13.97" size="1.778" layer="27" display="off"/>
@@
 <attribute name="PROD_ID" value=" " x="17.78" y="20.32" size="1.778" layer="27" rot="R180" display="off"/>
 </element>
-<element name="R56" library="SparkFun-Resistors" library_urn="urn:adsk.eagle:library:532" package="0603" package3d_urn="urn:adsk.eagle:package:39650/1" value=" 0" x="17.78" y="17.78" smashed="yes">
+<element name="R56" library="SparkFun-Resistors" library_urn="urn:adsk.eagle:library:532" package="0603" package3d_urn="urn:adsk.eagle:package:39650/1" value=" 100" x="17.78" y="17.78" smashed="yes">
 <attribute name="NAME" x="17.272" y="17.018" size="0.6096" layer="21" font="vector" ratio="13" rot="R180" align="bottom-center"/>
 <attribute name="PROD_ID" value=" " x="17.78" y="17.78" size="1.778" layer="27" display="off"/>
@@
 <attribute name="PROD_ID" value=" " x="10.16" y="11.43" size="1.778" layer="27" rot="R180" display="off"/>
 </element>
-<element name="R60" library="SparkFun-Resistors" library_urn="urn:adsk.eagle:library:532" package="0603" package3d_urn="urn:adsk.eagle:package:39650/1" value=" 0" x="10.16" y="8.89" smashed="yes">
+<element name="R60" library="SparkFun-Resistors" library_urn="urn:adsk.eagle:library:532" package="0603" package3d_urn="urn:adsk.eagle:package:39650/1" value=" 100" x="10.16" y="8.89" smashed="yes">
 <attribute name="NAME" x="9.652" y="8.128" size="0.6096" layer="21" font="vector" ratio="13" rot="R180" align="bottom-center"/>
 <attribute name="PROD_ID" value=" " x="10.16" y="8.89" size="1.778" layer="27" display="off"/>
@@
 <attribute name="PROD_ID" value=" " x="13.97" y="8.89" size="1.778" layer="27" display="off"/>
 </element>
-<element name="R57" library="SparkFun-Resistors" library_urn="urn:adsk.eagle:library:532" package="0603" package3d_urn="urn:adsk.eagle:package:39650/1" value=" 0" x="17.78" y="12.7" smashed="yes">
+<element name="R57" library="SparkFun-Resistors" library_urn="urn:adsk.eagle:library:532" package="0603" package3d_urn="urn:adsk.eagle:package:39650/1" value=" 100" x="17.78" y="12.7" smashed="yes">
 <attribute name="NAME" x="17.272" y="11.938" size="0.6096" layer="21" font="vector" ratio="13" rot="R180" align="bottom-center"/>
 <attribute name="PROD_ID" value=" " x="17.78" y="12.7" size="1.778" layer="27" display="off"/>
@@
 <attribute name="PROD_ID" value=" " x="21.59" y="12.7" size="1.778" layer="27" display="off"/>
 </element>
-<element name="R68" library="SparkFun-Resistors" library_urn="urn:adsk.eagle:library:532" package="0603" package3d_urn="urn:adsk.eagle:package:39650/1" value=" 0" x="17.78" y="7.62" smashed="yes">
+<element name="R68" library="SparkFun-Resistors" library_urn="urn:adsk.eagle:library:532" package="0603" package3d_urn="urn:adsk.eagle:package:39650/1" value=" 100" x="17.78" y="7.62" smashed="yes">
 <attribute name="NAME" x="17.272" y="6.858" size="0.6096" layer="21" font="vector" ratio="13" rot="R180" align="bottom-center"/>
 <attribute name="PROD_ID" value=" " x="17.78" y="7.62" size="1.778" layer="27" display="off"/>
@@
 <attribute name="PROD_ID" value=" " x="13.97" y="3.81" size="1.778" layer="27" display="off"/>
 </element>
-<element name="R69" library="SparkFun-Resistors" library_urn="urn:adsk.eagle:library:532" package="0603" package3d_urn="urn:adsk.eagle:package:39650/1" value=" 0" x="10.16" y="3.81" smashed="yes">
+<element name="R69" library="SparkFun-Resistors" library_urn="urn:adsk.eagle:library:532" package="0603" package3d_urn="urn:adsk.eagle:package:39650/1" value=" 100" x="10.16" y="3.81" smashed="yes">
 <attribute name="NAME" x="9.652" y="3.048" size="0.6096" layer="21" font="vector" ratio="13" rot="R180" align="bottom-center"/>
 <attribute name="PROD_ID" value=" " x="10.16" y="3.81" size="1.778" layer="27" display="off"/>
