File: PCBDesign/1.4Fv4/1.4Fv4.brd (EAGLE design)
At the start: 87.6 x 57.1 mm, 180 parts, among them U1 SN74LVC, U10 ISO7241, U11 PAM2305, U12 SN6501, U13 TRANSFO_3.3, U14 ADE9078, U15 PS2505, U16 SN74LVC, U17 PS2505, U2 PS2505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

Commit message: Updated BOM, changed schematic, and uploaded PDF of latest version under documents
Parts:
- R11, R12, R19, R20, R26, R27: value 2k -> 5k
Changed lines of the file:
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@@
 <attribute name="PROD_ID" value=" " x="85.09" y="23.114" size="1.778" layer="27" rot="R180" display="off"/>
 </element>
-<element name="R11" library="SparkFun-Resistors" library_urn="urn:adsk.eagle:library:532" package="0603" package3d_urn="urn:adsk.eagle:package:39650/1" value="2k" x="71.12" y="40.64" smashed="yes">
+<element name="R11" library="SparkFun-Resistors" library_urn="urn:adsk.eagle:library:532" package="0603" package3d_urn="urn:adsk.eagle:package:39650/1" value="5k" x="71.12" y="40.64" smashed="yes">
 <attribute name="NAME" x="71.12" y="41.402" size="0.6096" layer="21" font="vector" ratio="13" align="bottom-center"/>
 <attribute name="PROD_ID" value=" " x="71.12" y="40.64" size="1.778" layer="27" display="off"/>
 </element>
-<element name="R12" library="SparkFun-Resistors" library_urn="urn:adsk.eagle:library:532" package="0603" package3d_urn="urn:adsk.eagle:package:39650/1" value="2k" x="71.12" y="38.1" smashed="yes" rot="R180">
+<element name="R12" library="SparkFun-Resistors" library_urn="urn:adsk.eagle:library:532" package="0603" package3d_urn="urn:adsk.eagle:package:39650/1" value="5k" x="71.12" y="38.1" smashed="yes" rot="R180">
 <attribute name="NAME" x="71.12" y="38.862" size="0.6096" layer="21" font="vector" ratio="13" align="bottom-center"/>
 <attribute name="PROD_ID" value=" " x="71.12" y="38.1" size="1.778" layer="27" rot="R180" display="off"/>
@@
 <attribute name="PROD_ID" value=" " x="85.09" y="17.78" size="1.778" layer="27" rot="R180" display="off"/>
 </element>
-<element name="R19" library="SparkFun-Resistors" library_urn="urn:adsk.eagle:library:532" package="0603" package3d_urn="urn:adsk.eagle:package:39650/1" value="2k" x="71.12" y="34.29" smashed="yes">
+<element name="R19" library="SparkFun-Resistors" library_urn="urn:adsk.eagle:library:532" package="0603" package3d_urn="urn:adsk.eagle:package:39650/1" value="5k" x="71.12" y="34.29" smashed="yes">
 <attribute name="NAME" x="71.12" y="35.052" size="0.6096" layer="21" font="vector" ratio="13" align="bottom-center"/>
 <attribute name="PROD_ID" value=" " x="71.12" y="34.29" size="1.778" layer="27" display="off"/>
 </element>
-<element name="R20" library="SparkFun-Resistors" library_urn="urn:adsk.eagle:library:532" package="0603" package3d_urn="urn:adsk.eagle:package:39650/1" value="2k" x="71.12" y="31.75" smashed="yes" rot="R180">
+<element name="R20" library="SparkFun-Resistors" library_urn="urn:adsk.eagle:library:532" package="0603" package3d_urn="urn:adsk.eagle:package:39650/1" value="5k" x="71.12" y="31.75" smashed="yes" rot="R180">
 <attribute name="NAME" x="71.12" y="32.512" size="0.6096" layer="21" font="vector" ratio="13" align="bottom-center"/>
 <attribute name="PROD_ID" value=" " x="71.12" y="31.75" size="1.778" layer="27" rot="R180" display="off"/>
@@
 <attribute name="PROD_ID" value=" " x="85.09" y="12.446" size="1.778" layer="27" rot="R180" display="off"/>
 </element>
-<element name="R26" library="SparkFun-Resistors" library_urn="urn:adsk.eagle:library:532" package="0603" package3d_urn="urn:adsk.eagle:package:39650/1" value="2k" x="71.12" y="27.94" smashed="yes">
+<element name="R26" library="SparkFun-Resistors" library_urn="urn:adsk.eagle:library:532" package="0603" package3d_urn="urn:adsk.eagle:package:39650/1" value="5k" x="71.12" y="27.94" smashed="yes">
 <attribute name="NAME" x="71.12" y="28.702" size="0.6096" layer="21" font="vector" ratio="13" align="bottom-center"/>
 <attribute name="PROD_ID" value=" " x="71.12" y="27.94" size="1.778" layer="27" display="off"/>
 </element>
-<element name="R27" library="SparkFun-Resistors" library_urn="urn:adsk.eagle:library:532" package="0603" package3d_urn="urn:adsk.eagle:package:39650/1" value="2k" x="71.12" y="25.4" smashed="yes">
+<element name="R27" library="SparkFun-Resistors" library_urn="urn:adsk.eagle:library:532" package="0603" package3d_urn="urn:adsk.eagle:package:39650/1" value="5k" x="71.12" y="25.4" smashed="yes">
 <attribute name="NAME" x="71.12" y="26.162" size="0.6096" layer="21" font="vector" ratio="13" align="bottom-center"/>
 <attribute name="PROD_ID" value=" " x="71.12" y="25.4" size="1.778" layer="27" display="off"/>
